Commit message: re-write launch

File: smb_description/urdf/RS-16.urdf.xacro (robot description, xacro)
@@ -19,5 +19,5 @@
         <origin rpy="-1.5707 0 0" xyz="0 0 0"/>
         <geometry>
-          <mesh filename="package://robosense_description/meshes/robosense_16.dae" />
+          <mesh filename="package://smb_description/urdf/meshes/robosense_16.dae" />
         </geometry>
       </visual>
